Commit message: Calibrate baselink-camera

File: urdf/baselink-camera.urdf.xacro (robot description, xacro)
@@ -40,5 +40,5 @@
     <parent link="${namespace}/base_link" />
     <child link="${camera_link}" />
-    <origin xyz="0.08 0. -0.1578" rpy="0 0.27284641020683 0." />
+    <origin xyz="0.135 0.035 -0.105" rpy="0 0.52 0." />
   </joint>
 </robot>
